File: GiGaMega_universal_2/GiGaMega_universal_2.sch (EAGLE design)
At the start: 41 parts

Commit message: connect i2c devices
Parts:
- removed I2C_BMP: (no value), pinhead:PINHD-1X4
- added SPI1: (no value), pinhead:PINHD-1X6
- I2C_RTC: device pinhead:PINHD-1X4 -> pinhead:PINHD-1X5
- SPI_NRF24L: device pinhead:PINHD-1X6 -> pinhead:PINHD-1X7
Connections:
- new net SCL: I2C_OLED.3, I2C_RTC.3, JP2.21, SPI1.4
- new net SDA: I2C_OLED.4, I2C_RTC.4, JP2.22, SPI1.3
- net +5V: now also I2C_OLED.1, I2C_RTC.5, SPI1.6
- net GND: now also I2C_OLED.2, I2C_RTC.1, SPI1.5
Other:
- moved on the sheet: 315MHZ_IN, 315MHZ_OUT, 433MHZ_IN, 433MHZ_OUT, I2C_OLED, SPI, SPI_BMP
Changed lines of the file:
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@@
 <part name="C9" library="resistor" library_urn="urn:adsk.eagle:library:348" deviceset="C-EU" device="C1206K" package3d_urn="urn:adsk.eagle:package:26202/1" value="22mF/TNT"/>
 <part name="C10" library="resistor" library_urn="urn:adsk.eagle:library:348" deviceset="C-EU" device="C1206K" package3d_urn="urn:adsk.eagle:package:26202/1" value="22mF/TNT"/>
-<part name="I2C_BMP" library="pinhead" library_urn="urn:adsk.eagle:library:325" deviceset="PINHD-1X4" device="" package3d_urn="urn:adsk.eagle:package:22407/2"/>
-<part name="I2C_RTC" library="pinhead" library_urn="urn:adsk.eagle:library:325" deviceset="PINHD-1X4" device="" package3d_urn="urn:adsk.eagle:package:22407/2"/>
 <part name="I2C_OLED" library="pinhead" library_urn="urn:adsk.eagle:library:325" deviceset="PINHD-1X4" device="" package3d_urn="urn:adsk.eagle:package:22407/2"/>
-<part name="SPI_NRF24L" library="pinhead" library_urn="urn:adsk.eagle:library:325" deviceset="PINHD-1X6" device="" package3d_urn="urn:adsk.eagle:package:22472/2"/>
 <part name="SPI_BMP" library="pinhead" library_urn="urn:adsk.eagle:library:325" deviceset="PINHD-1X6" device="" package3d_urn="urn:adsk.eagle:package:22472/2"/>
 <part name="SPI" library="pinhead" library_urn="urn:adsk.eagle:library:325" deviceset="PINHD-1X6" device="" package3d_urn="urn:adsk.eagle:package:22472/2"/>
@@
 <part name="+3V2" library="supply1" library_urn="urn:adsk.eagle:library:371" deviceset="+3V3" device=""/>
 <part name="P+5" library="supply1" library_urn="urn:adsk.eagle:library:371" deviceset="+5V" device=""/>
+<part name="SPI_NRF24L" library="pinhead" library_urn="urn:adsk.eagle:library:325" deviceset="PINHD-1X7" device="" package3d_urn="urn:adsk.eagle:package:22477/2"/>
+<part name="P+6" library="supply1" library_urn="urn:adsk.eagle:library:371" deviceset="+5V" device=""/>
+<part name="GND5" library="supply1" library_urn="urn:adsk.eagle:library:371" deviceset="GND" device=""/>
+<part name="I2C_RTC" library="pinhead" library_urn="urn:adsk.eagle:library:325" deviceset="PINHD-1X5" device="" package3d_urn="urn:adsk.eagle:package:22469/2"/>
+<part name="P+7" library="supply1" library_urn="urn:adsk.eagle:library:371" deviceset="+5V" device=""/>
+<part name="GND6" library="supply1" library_urn="urn:adsk.eagle:library:371" deviceset="GND" device=""/>
+<part name="SPI1" library="pinhead" library_urn="urn:adsk.eagle:library:325" deviceset="PINHD-1X6" device="" package3d_urn="urn:adsk.eagle:package:22472/2"/>
 </parts>
 <sheets>
@@
 <instance part="P+4" gate="VCC" x="22.86" y="68.58"/>
 <instance part="GND4" gate="1" x="12.7" y="68.58" rot="R180"/>
-<instance part="I2C_BMP" gate="A" x="-5.08" y="7.62"/>
-<instance part="I2C_RTC" gate="A" x="7.62" y="7.62"/>
-<instance part="I2C_OLED" gate="A" x="-17.78" y="7.62"/>
-<instance part="SPI_NRF24L" gate="A" x="7.62" y="-22.86"/>
-<instance part="SPI_BMP" gate="A" x="-5.08" y="-22.86"/>
-<instance part="SPI" gate="A" x="-17.78" y="-22.86"/>
+<instance part="I2C_OLED" gate="A" x="127" y="127"/>
+<instance part="SPI_BMP" gate="A" x="-27.94" y="-15.24"/>
+<instance part="SPI" gate="A" x="-40.64" y="-15.24"/>
 <instance part="+5V" gate="A" x="7.62" y="-50.8"/>
 <instance part="DHT22" gate="A" x="43.18" y="-35.56" rot="R270"/>
@@
 <instance part="FLOW_H" gate="A" x="190.5" y="10.16"/>
 <instance part="TEMP_C" gate="A" x="190.5" y="30.48"/>
-<instance part="433MHZ_OUT" gate="A" x="40.64" y="116.84" rot="R90"/>
-<instance part="433MHZ_IN" gate="A" x="63.5" y="116.84" rot="R90"/>
-<instance part="315MHZ_OUT" gate="A" x="86.36" y="116.84" rot="R90"/>
-<instance part="315MHZ_IN" gate="A" x="109.22" y="116.84" rot="R90"/>
+<instance part="433MHZ_OUT" gate="A" x="-45.72" y="124.46" rot="R90"/>
+<instance part="433MHZ_IN" gate="A" x="-22.86" y="124.46" rot="R90"/>
+<instance part="315MHZ_OUT" gate="A" x="0" y="124.46" rot="R90"/>
+<instance part="315MHZ_IN" gate="A" x="22.86" y="124.46" rot="R90"/>
 <instance part="IR" gate="G$1" x="175.26" y="-35.56" rot="R270"/>
 <instance part="+3V3" gate="A" x="7.62" y="-66.04"/>
 <instance part="+3V2" gate="G$1" x="-10.16" y="-66.04" rot="R90"/>
 <instance part="P+5" gate="1" x="-10.16" y="-50.8" rot="R90"/>
+<instance part="SPI_NRF24L" gate="A" x="-15.24" y="-15.24"/>
+<instance part="P+6" gate="1" x="137.16" y="99.06"/>
+<instance part="GND5" gate="1" x="137.16" y="66.04"/>
+<instance part="I2C_RTC" gate="A" x="127" y="81.28" rot="R180"/>
+<instance part="P+7" gate="1" x="127" y="144.78" rot="R270"/>
+<instance part="GND6" gate="1" x="104.14" y="144.78" rot="R270"/>
+<instance part="SPI1" gate="A" x="127" y="165.1"/>
 </instances>
 <busses>
@@
 <junction x="43.18" y="55.88"/>
 </segment>
+<segment>
+<pinref part="GND5" gate="1" pin="GND"/>
+<wire x1="137.16" y1="68.58" x2="137.16" y2="76.2" width="0.1524" layer="91"/>
+<pinref part="I2C_RTC" gate="A" pin="1"/>
+<wire x1="129.54" y1="76.2" x2="137.16" y2="76.2" width="0.1524" layer="91"/>
+</segment>
+<segment>
+<pinref part="I2C_OLED" gate="A" pin="2"/>
+<wire x1="124.46" y1="129.54" x2="111.76" y2="129.54" width="0.1524" layer="91"/>
+<pinref part="GND6" gate="1" pin="GND"/>
+<wire x1="111.76" y1="129.54" x2="111.76" y2="144.78" width="0.1524" layer="91"/>
+<wire x1="111.76" y1="144.78" x2="106.68" y2="144.78" width="0.1524" layer="91"/>
+<wire x1="111.76" y1="144.78" x2="111.76" y2="162.56" width="0.1524" layer="91"/>
+<pinref part="SPI1" gate="A" pin="5"/>
+<wire x1="111.76" y1="162.56" x2="124.46" y2="162.56" width="0.1524" layer="91"/>
+<junction x="111.76" y="144.78"/>
+</segment>
 </net>
 <net name="+3V3" class="0">
@@
 <pinref part="P+5" gate="1" pin="+5V"/>
 </segment>
-</net>
+<segment>
+<pinref part="P+6" gate="1" pin="+5V"/>
+<wire x1="137.16" y1="86.36" x2="137.16" y2="96.52" width="0.1524" layer="91"/>
+<pinref part="I2C_RTC" gate="A" pin="5"/>
+<wire x1="129.54" y1="86.36" x2="137.16" y2="86.36" width="0.1524" layer="91"/>
+</segment>
+<segment>
+<pinref part="I2C_OLED" gate="A" pin="1"/>
+<wire x1="124.46" y1="132.08" x2="116.84" y2="132.08" width="0.1524" layer="91"/>
+<wire x1="116.84" y1="132.08" x2="116.84" y2="144.78" width="0.1524" layer="91"/>
+<pinref part="SPI1" gate="A" pin="6"/>
+<wire x1="116.84" y1="144.78" x2="116.84" y2="160.02" width="0.1524" layer="91"/>
+<wire x1="116.84" y1="160.02" x2="124.46" y2="160.02" width="0.1524" layer="91"/>
+<pinref part="P+7" gate="1" pin="+5V"/>
+<wire x1="124.46" y1="144.78" x2="116.84" y2="144.78" width="0.1524" layer="91"/>
+<junction x="116.84" y="144.78"/>
+</segment>
+</net>
+<net name="SDA" class="0">
+<segment>
+<pinref part="JP2" gate="A" pin="22"/>
+<wire x1="132.08" y1="25.4" x2="144.78" y2="25.4" width="0.1524" layer="91"/>
+<pinref part="I2C_RTC" gate="A" pin="4"/>
+<wire x1="144.78" y1="25.4" x2="144.78" y2="83.82" width="0.1524" layer="91"/>
+<wire x1="144.78" y1="83.82" x2="129.54" y2="83.82" width="0.1524" layer="91"/>
+<label x="144.78" y="71.12" size="1.778" layer="95"/>
+<pinref part="I2C_OLED" gate="A" pin="4"/>
+<wire x1="144.78" y1="83.82" x2="144.78" y2="124.46" width="0.1524" layer="91"/>
+<wire x1="144.78" y1="124.46" x2="124.46" y2="124.46" width="0.1524" layer="91"/>
+<pinref part="SPI1" gate="A" pin="3"/>
+<wire x1="144.78" y1="124.46" x2="144.78" y2="167.64" width="0.1524" layer="91"/>
+<wire x1="144.78" y1="167.64" x2="124.46" y2="167.64" width="0.1524" layer="91"/>
+</segment>
+</net>
+<net name="SCL" class="0">
+<segment>
+<pinref part="JP2" gate="A" pin="21"/>
+<wire x1="124.46" y1="25.4" x2="114.3" y2="25.4" width="0.1524" layer="91"/>
+<wire x1="114.3" y1="25.4" x2="114.3" y2="81.28" width="0.1524" layer="91"/>
+<pinref part="I2C_RTC" gate="A" pin="3"/>
+<wire x1="129.54" y1="81.28" x2="114.3" y2="81.28" width="0.1524" layer="91"/>
+<label x="114.3" y="58.42" size="1.778" layer="95"/>
+<pinref part="I2C_OLED" gate="A" pin="3"/>
+<wire x1="114.3" y1="81.28" x2="114.3" y2="127" width="0.1524" layer="91"/>
+<wire x1="114.3" y1="127" x2="124.46" y2="127" width="0.1524" layer="91"/>
+<wire x1="114.3" y1="127" x2="99.06" y2="127" width="0.1524" layer="91"/>
+<pinref part="SPI1" gate="A" pin="4"/>
+<wire x1="99.06" y1="127" x2="99.06" y2="165.1" width="0.1524" layer="91"/>
+<wire x1="99.06" y1="165.1" x2="124.46" y2="165.1" width="0.1524" layer="91"/>
+</segment>
+</net>

Commit message: changed power board
Parts:
- added C11, C12, C13: (no value), rcl:CPOL-USUD-6,3X7,7
- added C14, C15, C16: TAJD107K020RNJTAJD-M, capacitor_tantal:TAJD107K020RNJTAJD-M
- added CR1, CR2, CR3: SS32-E3/57TDIODE_DO214AB-M, SS32:SS32-E3/57TDIODE_DO214AB-M
- added IC1, IC2, IC3: LM2596S, national-semiconductor:LM2596S
- added R1, R2, R3, R4, R5, R6: (no value), rcl:R-EU_R1206
Changed lines of the file:
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@@
 <part name="GND6" library="supply1" library_urn="urn:adsk.eagle:library:371" deviceset="GND" device=""/>
 <part name="SPI1" library="pinhead" library_urn="urn:adsk.eagle:library:325" deviceset="PINHD-1X6" device="" package3d_urn="urn:adsk.eagle:package:22472/2"/>
+<part name="C11" library="rcl" library_urn="urn:adsk.eagle:library:334" deviceset="CPOL-US" device="UD-6,3X7,7" package3d_urn="urn:adsk.eagle:package:23472/1"/>
+<part name="C12" library="rcl" library_urn="urn:adsk.eagle:library:334" deviceset="CPOL-US" device="UD-6,3X7,7" package3d_urn="urn:adsk.eagle:package:23472/1"/>
+<part name="C13" library="rcl" library_urn="urn:adsk.eagle:library:334" deviceset="CPOL-US" device="UD-6,3X7,7" package3d_urn="urn:adsk.eagle:package:23472/1"/>
+<part name="CR1" library="SS32" deviceset="SS32-E3/57T" device="DIODE_DO214AB-M"/>
+<part name="CR2" library="SS32" deviceset="SS32-E3/57T" device="DIODE_DO214AB-M"/>
+<part name="CR3" library="SS32" deviceset="SS32-E3/57T" device="DIODE_DO214AB-M"/>
+<part name="C14" library="capacitor_tantal" deviceset="TAJD107K020RNJ" device="TAJD-M"/>
+<part name="C15" library="capacitor_tantal" deviceset="TAJD107K020RNJ" device="TAJD-M"/>
+<part name="C16" library="capacitor_tantal" deviceset="TAJD107K020RNJ" device="TAJD-M"/>
+<part name="IC1" library="national-semiconductor" library_urn="urn:adsk.eagle:library:307" deviceset="LM2596" device="S" package3d_urn="urn:adsk.eagle:package:21218/1"/>
+<part name="IC2" library="national-semiconductor" library_urn="urn:adsk.eagle:library:307" deviceset="LM2596" device="S" package3d_urn="urn:adsk.eagle:package:21218/1"/>
+<part name="IC3" library="national-semiconductor" library_urn="urn:adsk.eagle:library:307" deviceset="LM2596" device="S" package3d_urn="urn:adsk.eagle:package:21218/1"/>
+<part name="R1" library="rcl" library_urn="urn:adsk.eagle:library:334" deviceset="R-EU_" device="R1206" package3d_urn="urn:adsk.eagle:package:23540/2"/>
+<part name="R2" library="rcl" library_urn="urn:adsk.eagle:library:334" deviceset="R-EU_" device="R1206" package3d_urn="urn:adsk.eagle:package:23540/2"/>
+<part name="R3" library="rcl" library_urn="urn:adsk.eagle:library:334" deviceset="R-EU_" device="R1206" package3d_urn="urn:adsk.eagle:package:23540/2"/>
+<part name="R4" library="rcl" library_urn="urn:adsk.eagle:library:334" deviceset="R-EU_" device="R1206" package3d_urn="urn:adsk.eagle:package:23540/2"/>
+<part name="R5" library="rcl" library_urn="urn:adsk.eagle:library:334" deviceset="R-EU_" device="R1206" package3d_urn="urn:adsk.eagle:package:23540/2"/>
+<part name="R6" library="rcl" library_urn="urn:adsk.eagle:library:334" deviceset="R-EU_" device="R1206" package3d_urn="urn:adsk.eagle:package:23540/2"/>
 </parts>
 <sheets>
@@
 <instance part="C9" gate="G$1" x="71.12" y="58.42"/>
 <instance part="C10" gate="G$1" x="129.54" y="58.42"/>
+<instance part="C11" gate="G$1" x="40.64" y="17.78"/>
+<instance part="C12" gate="G$1" x="114.3" y="-2.54"/>
+<instance part="C13" gate="G$1" x="152.4" y="50.8"/>
+<instance part="CR1" gate="A" x="30.48" y="-7.62"/>
+<instance part="CR2" gate="A" x="109.22" y="-20.32"/>
+<instance part="CR3" gate="A" x="165.1" y="45.72"/>
+<instance part="C14" gate="A" x="25.4" y="-22.86"/>
+<instance part="C15" gate="A" x="111.76" y="-38.1"/>
+<instance part="C16" gate="A" x="177.8" y="27.94"/>
+<instance part="IC1" gate="G$1" x="22.86" y="88.9"/>
+<instance part="IC2" gate="G$1" x="96.52" y="93.98"/>
+<instance part="IC3" gate="G$1" x="160.02" y="-2.54"/>
+<instance part="R1" gate="G$1" x="53.34" y="40.64" rot="R90"/>
+<instance part="R2" gate="G$1" x="53.34" y="25.4" rot="R90"/>
+<instance part="R3" gate="G$1" x="177.8" y="60.96" rot="R90"/>
+<instance part="R4" gate="G$1" x="190.5" y="60.96" rot="R90"/>
+<instance part="R5" gate="G$1" x="195.58" y="-7.62" rot="R90"/>
+<instance part="R6" gate="G$1" x="195.58" y="-20.32" rot="R90"/>
 </instances>
 <busses>
@@
 packages will not be understood (or retained) with this version.
 </note>
+<note version="8.4" severity="warning">
+Since Version 8.4, EAGLE supports properties for SPICE simulation.
+Probes in schematics and SPICE mapping objects found in parts and library devices
+will not be understood with this version. Update EAGLE to the latest version
+for full support of SPICE simulation.
+</note>
 </compatibility>
