File: GiGaMega_universal_2/GiGaMega_universal_2.sch (EAGLE design)
At the start: 49 parts, among them IC1 LM2596S, IC2 LM2596S, IC4 LM2596S

Commit message: added sensors connection
Parts:
- removed JP4: (no value), pinhead:PINHD-2X3
- removed SPI1: (no value), pinhead:PINHD-1X6
- added I2C_BMP280: (no value), pinhead:PINHD-1X6
- added SPI_NRF24L_2: (no value), pinhead:PINHD-2X4
- AIR: device pinhead:PINHD-1X3 -> pinhead:PINHD-1X4
Connections:
- new net D5: +5V.1, +5V.2, +5V.3, AIR.2, AIR.4, C2.2, DHT22.1, FLOW_C.2, FLOW_H.2, I2C_BMP280.6, I2C_OLED.1, I2C_RTC.5, JP1.13, L2.2, R7.2, TEMP_C.2, TEMP_H.2
- new net INT2(D19): FLOW_H.3, JP1.27
- new net INT3(D18): FLOW_C.3, JP1.28
- new net N$7: JP1.31, TEMP_H.3
- new net N$8: JP1.32, TEMP_C.3
- new net N$9: DHT22.2, JP1.14
- net +3V3: now also SPI_NRF24L.6, SPI_NRF24L_2.8
- net +5V: now also AIR.1, JP1.11, JP1.16, JP2.2, JP2.29, JP2.30, JP2.31, JP2.32, MOOW.1, MOOW.2, SPI_NRF24L_2.1, SPI_NRF24L_2.3, SPI_NRF24L_2.4, SPI_NRF24L_2.5, SPI_NRF24L_2.6; no longer +5V.1, +5V.2, +5V.3, C2.2, I2C_OLED.1, I2C_RTC.5, L2.2, R7.2, SPI1.6
- net GND: now also AIR.3, DHT22.3, FLOW_C.1, FLOW_H.1, I2C_BMP280.5, MOOW.3, SPI_NRF24L.7, SPI_NRF24L_2.7, TEMP_C.1, TEMP_H.1; no longer SPI1.5
- net SCL: now also I2C_BMP280.4, JP1.29; no longer JP2.21, SPI1.4
- net SDA: now also I2C_BMP280.3, JP1.30; no longer JP2.22, SPI1.3
Other:
- moved on the sheet: +3V3, +5V, 315MHZ_IN, 315MHZ_OUT, 433MHZ_IN, 433MHZ_OUT, DHT22, FLOW_C, FLOW_H, I2C_OLED, I2C_RTC, IR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

Commit message: add IR, LIGHT 433, 315 sensors
Parts:
- added R5: 4.7k, eagle-ltspice:RR1206
- added R6: 470, eagle-ltspice:RR1206
- added T1: 2N2222, transistor:2N2222
- LIGHT: device pinhead:PINHD-1X3 -> pinhead:PINHD-1X2
Connections:
- new net N$10: IR.1, T1.C
- new net N$11: R6.1, T1.B
- net +5V: now also 315MHZ_IN.2, 315MHZ_IN.3, 315MHZ_IN.4, 315MHZ_OUT.2, 315MHZ_OUT.3, 315MHZ_OUT.4, 433MHZ_IN.2, 433MHZ_IN.3, 433MHZ_IN.4, 433MHZ_OUT.2, 433MHZ_OUT.3, 433MHZ_OUT.4, IR.2, JP2.1, KEYBOARD.2, KEYBOARD.3, LIGHT.1, LIGHT.2, R5.2, R6.2
- net GND: now also 315MHZ_IN.1, 315MHZ_OUT.1, 433MHZ_IN.1, 433MHZ_OUT.1, KEYBOARD.1, R5.1, T1.E
Other:
- moved on the sheet: 315MHZ_IN, 315MHZ_OUT, 433MHZ_IN, 433MHZ_OUT, IR, KEYBOARD

Commit message: added all sensors
Parts:
- removed JP21: (no value), pinhead:PINHD-1X3
- removed JP3: (no value), pinhead:PINHD-2X3
- removed JP5: (no value), pinhead:PINHD-1X5
- removed SPI_BMP: (no value), pinhead:PINHD-1X6
- removed T1: 2N2222, transistor:2N2222
- R6: value 470 -> 300
Connections:
- removed net N$10: IR.1, T1.C
- net +5V: now also JP1.15, JP1.17, JP1.18, JP1.19, JP1.20, R6.1, SPI.1, SPI.2, SPI.3, SPI.4, SPI.5, SPI_NRF24L.1, SPI_NRF24L.2, SPI_NRF24L.3, SPI_NRF24L.4, SPI_NRF24L.5; no longer IR.2, R6.2
- net GND: now also IR.1, SPI.6; no longer T1.E
- net N$11: now also IR.2, R6.2; no longer R6.1, T1.B
Other:
- moved on the sheet: R6
